File: I2C-Oled-Backpack-EastRising.brd (EAGLE design)
At the start: 41.9 x 19.1 mm, 14 parts, among them J1 4P-SMD-2.0-90D, J2 4P-SMD-2.0-90D, J3 15P-2.54

Commit message: Rev D
Other:
- board text added: "(Rev D)"
- board text added: "I2C OLED Backpack (ER) (Rev D)"
- board text added: "dcity.org"
- board text removed: "(Rev C)"
- board text removed: "I2C OLED Backpack (ER) (Rev C)"
- board text removed: "wht.io"
Changed lines of the file:
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@@
 <?xml version="1.0" encoding="utf-8"?>
 <!DOCTYPE eagle SYSTEM "eagle.dtd">
-<eagle version="7.5.0">
+<eagle version="9.1.3">
 <drawing>
 <settings>
 <setting alwaysvectorfont="no"/>
+<setting keepoldvectorfont="yes"/>
 <setting verticaltext="up"/>
 </settings>
 <grid distance="0.05" unitdist="inch" unit="inch" style="lines" multiple="1" display="yes" altdistance="0.005" altunitdist="inch" altunit="inch"/>
 <layers>
-<layer number="1" name="Top" color="4" fill="1" visible="yes" active="yes"/>
-<layer number="16" name="Bottom" color="1" fill="1" visible="yes" active="yes"/>
-<layer number="17" name="Pads" color="2" fill="1" visible="yes" active="yes"/>
-<layer number="18" name="Vias" color="2" fill="1" visible="yes" active="yes"/>
-<layer number="19" name="Unrouted" color="6" fill="1" visible="yes" active="yes"/>
+<layer number="1" name="Top" color="4" fill="1" visible="no" active="yes"/>
+<layer number="16" name="Bottom" color="1" fill="1" visible="no" active="yes"/>
+<layer number="17" name="Pads" color="2" fill="1" visible="no" active="yes"/>
+<layer number="18" name="Vias" color="2" fill="1" visible="no" active="yes"/>
+<layer number="19" name="Unrouted" color="6" fill="1" visible="no" active="yes"/>
 <layer number="20" name="Dimension" color="15" fill="1" visible="yes" active="yes"/>
-<layer number="21" name="tPlace" color="7" fill="1" visible="yes" active="yes"/>
-<layer number="22" name="bPlace" color="7" fill="1" visible="yes" active="yes"/>
+<layer number="21" name="tPlace" color="7" fill="1" visible="no" active="yes"/>
+<layer number="22" name="bPlace" color="7" fill="1" visible="no" active="yes"/>
 <layer number="23" name="tOrigins" color="15" fill="1" visible="yes" active="yes"/>
 <layer number="24" name="bOrigins" color="15" fill="1" visible="yes" active="yes"/>
@@
 <text x="27.7876" y="17.7038" size="0.889" layer="21" font="vector" ratio="11">I2C OLED BKPK (ER)</text>
 <text x="23.8506" y="18.1356" size="0.889" layer="21" font="vector" ratio="11">+</text>
-<text x="40.64" y="17.145" size="0.889" layer="22" font="vector" ratio="11" rot="MR0">I2C OLED Backpack (ER) (Rev C)</text>
+<text x="40.64" y="17.145" size="0.889" layer="22" font="vector" ratio="11" rot="MR0">I2C OLED Backpack (ER) (Rev D)</text>
 <text x="19.558" y="3.048" size="0.889" layer="21" font="vector" ratio="11" rot="R90">SDA</text>
 <text x="14.351" y="3.048" size="0.889" layer="21" font="vector" ratio="11" rot="R90">SCL</text>
 <text x="37.338" y="2.921" size="0.889" layer="21" font="vector" ratio="11" rot="R90">G</text>
 <text x="34.671" y="2.921" size="0.889" layer="21" font="vector" ratio="11" rot="R90">V</text>
-<text x="1.524" y="16.9418" size="1.524" layer="21" font="vector" ratio="10">wht.io</text>
+<text x="1.524" y="16.9418" size="1.524" layer="21" font="vector" ratio="10">dcity.org</text>
 <rectangle x1="13.0556" y1="13.8176" x2="14.732" y2="15.0114" layer="43"/>
 <rectangle x1="15.621" y1="13.7922" x2="17.2212" y2="15.0622" layer="43"/>
@@
 <rectangle x1="29.5402" y1="14.1986" x2="31.3436" y2="15.7734" layer="43"/>
 <rectangle x1="10.4648" y1="14.4018" x2="12.5984" y2="15.8496" layer="43"/>
-<text x="7.747" y="16.891" size="1.524" layer="22" font="vector" ratio="10" rot="MR0">wht.io</text>
-<text x="27.813" y="16.637" size="0.889" layer="21" font="vector" ratio="11">(Rev C)</text>
+<text x="11.557" y="16.891" size="1.524" layer="22" font="vector" ratio="10" rot="MR0">dcity.org</text>
+<text x="27.813" y="16.637" size="0.889" layer="21" font="vector" ratio="11">(Rev D)</text>
 <text x="15.24" y="11.43" size="0.889" layer="21" font="vector" ratio="11">C=3C</text>
 <text x="15.24" y="12.573" size="0.889" layer="21" font="vector" ratio="11">O=3D</text>
+<wire x1="41.91" y1="19.05" x2="41.91" y2="0" width="0" layer="20"/>
 </plain>
 <attributes>
@@
 <param name="dpMaxLengthDifference" value="10mm"/>
 <param name="dpGapFactor" value="2.5"/>
-<param name="checkGrid" value="0"/>
 <param name="checkAngle" value="1"/>
 <param name="checkFont" value="1"/>
 <param name="checkRestrict" value="1"/>
+<param name="checkStop" value="0"/>
+<param name="checkValues" value="0"/>
+<param name="checkNames" value="1"/>
+<param name="checkWireStubs" value="1"/>
+<param name="checkPolygonWidth" value="0"/>
 <param name="useDiameter" value="13"/>
 <param name="maxErrors" value="50"/>
@@
 </signal>
 </signals>
+<mfgpreviewcolors>
+<mfgpreviewcolor name="soldermaskcolor" color="0xC8008000"/>
+<mfgpreviewcolor name="silkscreencolor" color="0xFFFEFEFE"/>
+<mfgpreviewcolor name="backgroundcolor" color="0xFF282828"/>
+<mfgpreviewcolor name="coppercolor" color="0xFFFFBF00"/>
+<mfgpreviewcolor name="substratecolor" color="0xFF786E46"/>
+</mfgpreviewcolors>
 </board>
 </drawing>

Commit message: Rev E
Parts:
- J1, J2: value 4P-SMD-2.0-90D -> QWIIC_RIGHT_ANGLE; device 0:HW4-SMD-2.0-90D -> 0:JST04_1MM_RA
- moved J1 26.8 mm to (4.95, 9.53)
- moved J2 26.7 mm to (36.8, 9.53)
Connections:
- net GND: now also J1.1, J2.1; no longer J1.4, J2.4
- net SCL: now also J1.4, J2.4; no longer J1.1, J2.1
- net SDA: now also J1.3, J2.3; no longer J1.2, J2.2
- net VCC: now also J1.2, J2.2; no longer J1.3, J2.3
Routing:
- net SDA: track 55.8 -> 72.3 mm
- net SCL: track 29.9 -> 42.3 mm
- net VCC: track 58.9 -> 64.9 mm
- net SA0: track 22.9 -> 19.9 mm, vias 0 -> 2
- net RES: track 22.7 -> 20.4 mm
Other:
- board text added: "(Rev E)"
- board text added: "I2C OLED Backpack (ER) (Rev E)"
- board text removed: "(Rev D)"
- board text removed: "I2C OLED Backpack (ER) (Rev D)"
